File: docs/pcb/PCB.kicad_sch (KiCad schematic)
At the start: 82 parts, among them J1 Screw_Terminal_01x02, J2 Screw_Terminal_01x03, J3 Screw_Terminal_01x07, J4 Screw_Terminal_01x02, J5 Screw_Terminal_01x02, J6 Screw_Terminal_01x04, J7 Screw_Terminal_01x02, J8 Screw_Terminal_01x07, Q1 BC109, Q2 BC109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

Commit message: Schematic and materials update
Parts:
- R1, R13, R21, R4, R5, R6, R9: value 1.1k -> 33k
